Commit message: update

File: workspace/ros2_ws/src/opencr_hardware/urdf/opencr.ros2_control.xacro (robot description, xacro)
@@ -27,10 +27,10 @@
     </joint>
   </xacro:macro>
-  <!-- wheel_count: 4 (기본, waffle_4wd) 또는 6 -->
-  <xacro:macro name="opencr_ros2_control" params="name:=OpenCRSystem port:=/dev/opencr wheel_count:=4 use_gripper:=false joy_required:=true">
+  <!-- 두 OpenCR의 순서는 고정하지 않고 STATE.role로 역할을 판별한다. -->
+  <xacro:macro name="opencr_ros2_control" params="name:=OpenCRSystem ports:=/dev/ttyACM0,/dev/ttyACM1 wheel_count:=6 use_gripper:=false joy_required:=true">
     <ros2_control name="${name}" type="system">
       <hardware>
         <plugin>opencr_hardware/OpenCRHardware</plugin>
-        <param name="port">${port}</param>
+        <param name="ports">${ports}</param>
         <param name="comm_timeout_s">0.5</param>
         <param name="first_state_timeout_s">2.0</param>

File: workspace/ros2_ws/src/opencr_hardware/urdf/robot.urdf.xacro (robot description, xacro)
@@ -4,7 +4,7 @@
      형상(visual/collision)은 넣지 않았다. waffle_4wd 메시를 쓰려면 base_link 에 visual 을 추가한다. -->
 <robot name="puckbot" xmlns:xacro="http://www.ros.org/wiki/xacro">
-  <xacro:arg name="wheel_count" default="4"/>
+  <xacro:arg name="wheel_count" default="6"/>
   <xacro:arg name="use_gripper" default="false"/>
-  <xacro:arg name="port" default="/dev/opencr"/>
+  <xacro:arg name="ports" default="/dev/ttyACM0,/dev/ttyACM1"/>
   <xacro:arg name="joy_required" default="true"/>
   <xacro:include filename="$(find opencr_hardware)/urdf/opencr.ros2_control.xacro"/>
@@ -66,5 +66,5 @@
   <xacro:fixed_link name="tfmini_link"     parent="gripper_roll_link" xyz="0.02 0 -0.035" rpy="0 0 0"/>
   <xacro:fixed_link name="tool_link"       parent="gripper_roll_link" xyz="0.086 0 0" rpy="0 0 0"/>
-  <xacro:opencr_ros2_control port="$(arg port)" wheel_count="${wheel_count}" use_gripper="$(arg use_gripper)"
+  <xacro:opencr_ros2_control ports="$(arg ports)" wheel_count="${wheel_count}" use_gripper="$(arg use_gripper)"
                              joy_required="$(arg joy_required)"/>
 </robot>
