Commit message: feat: switch drive to 4 wheels and split firmware build by role
Co-Authored-By: Claude Opus 5.5 <noreply@anthropic.com>

File: workspace/ros2_ws/src/opencr_hardware/urdf/opencr.ros2_control.xacro (robot description, xacro)
@@ -28,5 +28,6 @@
   </xacro:macro>
   <!-- 두 OpenCR의 순서는 고정하지 않고 STATE.role로 역할을 판별한다. -->
-  <xacro:macro name="opencr_ros2_control" params="name:=OpenCRSystem ports:=/dev/ttyACM0,/dev/ttyACM1 wheel_count:=6 use_gripper:=false joy_required:=true">
+  <!-- wheel_count 4 의 칸 순서 (왼앞 0 · 왼뒤 1 · 오른앞 2 · 오른뒤 3) 는 주행 펌웨어 config.h WHEEL_IDS · WHEEL_DIR 와 같다 -->
+  <xacro:macro name="opencr_ros2_control" params="name:=OpenCRSystem ports:=/dev/ttyACM0,/dev/ttyACM1 wheel_count:=4 use_gripper:=false joy_required:=true">
     <ros2_control name="${name}" type="system">
       <hardware>

File: workspace/ros2_ws/src/opencr_hardware/urdf/robot.urdf.xacro (robot description, xacro)
@@ -4,5 +4,5 @@
      형상(visual/collision)은 넣지 않았다. waffle_4wd 메시를 쓰려면 base_link 에 visual 을 추가한다. -->
 <robot name="puckbot" xmlns:xacro="http://www.ros.org/wiki/xacro">
-  <xacro:arg name="wheel_count" default="6"/>
+  <xacro:arg name="wheel_count" default="4"/>   <!-- 주행 펌웨어 WHEEL_COUNT 와 같게 (2026-10-26 가운데 2개 제거) -->
   <xacro:arg name="use_gripper" default="false"/>
   <xacro:arg name="ports" default="/dev/ttyACM0,/dev/ttyACM1"/>

Commit message: feat: switch URDF to cartridar_01 CAD model
Co-Authored-By: Claude Opus 5.5 <noreply@anthropic.com>

File: workspace/ros2_ws/src/opencr_hardware/urdf/opencr.ros2_control.xacro (robot description, xacro)
@@ -1,6 +1,6 @@
 <?xml version="1.0"?>
 <!-- OpenCRHardware ros2_control 블록 (Firmware 팀).
-     바퀴 슬롯 = 펌웨어 config.h 의 WHEEL_IDS 순서 (왼쪽 앞→뒤, 오른쪽 앞→뒤).
-     팔 슬롯 0~5 = ARM_IDS 11~16 (joint1~5, gripper_roll). -->
+     바퀴 칸 0~3 = 주행 펌웨어 config.h 의 WHEEL_IDS 순서 (왼쪽 앞 · 왼쪽 뒤 · 오른쪽 앞 · 오른쪽 뒤).
+     팔 칸 0~5 = 팔 펌웨어 ARM_IDS 순서 (joint1~4 · wrist_roll_joint · gripper_motor_joint). -->
 <robot xmlns:xacro="http://www.ros.org/wiki/xacro">
   <xacro:macro name="opencr_wheel" params="name slot">
@@ -28,6 +28,7 @@
   </xacro:macro>
   <!-- 두 OpenCR의 순서는 고정하지 않고 STATE.role로 역할을 판별한다. -->
-  <!-- wheel_count 4 의 칸 순서 (왼앞 0 · 왼뒤 1 · 오른앞 2 · 오른뒤 3) 는 주행 펌웨어 config.h WHEEL_IDS · WHEEL_DIR 와 같다 -->
-  <xacro:macro name="opencr_ros2_control" params="name:=OpenCRSystem ports:=/dev/ttyACM0,/dev/ttyACM1 wheel_count:=4 use_gripper:=false joy_required:=true">
+  <!-- 관절 이름은 CAD URDF (cartridar_01.urdf) 와 같다. 바퀴 칸 (왼앞 0 · 왼뒤 1 · 오른앞 2 · 오른뒤 3) 은 주행 펌웨어 config.h WHEEL_IDS ·
+       WHEEL_DIR 와, 팔 칸 0~5 는 팔 펌웨어 ARM_IDS {11, 12, 13, 16, 14, 15} 순서와 같다. -->
+  <xacro:macro name="opencr_ros2_control" params="name:=OpenCRSystem ports:=/dev/ttyACM0,/dev/ttyACM1 joy_required:=true">
     <ros2_control name="${name}" type="system">
       <hardware>
@@ -44,33 +45,24 @@
         <param name="battery_error_v">10.5</param>
       </hardware>
-      <xacro:if value="${wheel_count == 4}">
-        <xacro:opencr_wheel name="wheel_left_front_joint"  slot="0"/>
-        <xacro:opencr_wheel name="wheel_left_rear_joint"   slot="1"/>
-        <xacro:opencr_wheel name="wheel_right_front_joint" slot="2"/>
-        <xacro:opencr_wheel name="wheel_right_rear_joint"  slot="3"/>
-      </xacro:if>
-      <xacro:if value="${wheel_count == 6}">
-        <xacro:opencr_wheel name="wheel_left_front_joint"  slot="0"/>
-        <xacro:opencr_wheel name="wheel_left_mid_joint"    slot="1"/>
-        <xacro:opencr_wheel name="wheel_left_rear_joint"   slot="2"/>
-        <xacro:opencr_wheel name="wheel_right_front_joint" slot="3"/>
-        <xacro:opencr_wheel name="wheel_right_mid_joint"   slot="4"/>
-        <xacro:opencr_wheel name="wheel_right_rear_joint"  slot="5"/>
-      </xacro:if>
-      <!-- 관절 한계 (rad) — manipulator.yaml 의 joint_limits 와 맞춤 ★ 실측 -->
-      <xacro:opencr_arm_joint name="joint1"       slot="0" lower="-2.8" upper="2.8"/>
-      <xacro:opencr_arm_joint name="joint2"       slot="1" lower="-1.8" upper="1.6"/>
-      <xacro:opencr_arm_joint name="joint3"       slot="2" lower="-1.6" upper="1.5"/>
-      <xacro:opencr_arm_joint name="joint4"       slot="3" lower="-1.8" upper="2.0"/>
-      <xacro:opencr_arm_joint name="joint5"       slot="4" lower="-2.8" upper="2.8"/>
-      <xacro:opencr_arm_joint name="gripper_roll" slot="5" lower="-2.8" upper="2.8"/>
-      <xacro:if value="${use_gripper}">
-        <!-- 그리퍼 개폐 액추에이터 미정 — 정해지면 펌웨어 GRIPPER_ID 와 함께 켬 ★ -->
-        <joint name="gripper_joint">
-          <param name="role">gripper</param>
-          <command_interface name="position"/>
-          <state_interface name="position"/>
-        </joint>
-      </xacro:if>
+      <xacro:opencr_wheel name="wheel_fl_joint" slot="0"/>
+      <xacro:opencr_wheel name="wheel_rl_joint" slot="1"/>
+      <xacro:opencr_wheel name="wheel_fr_joint" slot="2"/>
+      <xacro:opencr_wheel name="wheel_rr_joint" slot="3"/>
+      <!-- 팔 관절 한계 (rad): 호스트가 명령을 이 범위로 자른다 = URDF 한계와 펌웨어 config.h ARM_MIN/MAX_RAD 가 겹치는 구간
+           (펌웨어는 범위 밖 CMD 를 통째로 거부하므로 넘으면 안 됨 - test_robot_description 이 확인).
+           URDF (cartridar_01) 는 보관함 계획 값 J1 ±π · J4 위 2.164 라 joint1 · joint4 는 펌웨어 범위 (±2.8 · 2.0) 에서 잘림.
+           보관함 앞 줄 (J1 최대 2.98 · J4 최대 2.16) 을 쓰려면 펌웨어 범위 · 모터 EEPROM 위치 한계를 넓힌 뒤 (장치 쓰기, 승인) 여기도 넓힘 ★.
+           기구 간섭 (홈 자세 J1 > 137° 면 뒤 프로파일, 롤 180° 근처 J4 > 112° 면 카메라) 은 경로 계획이 피해야 함 -->
+      <xacro:opencr_arm_joint name="joint1"           slot="0" lower="-2.8"    upper="2.8"/>
+      <xacro:opencr_arm_joint name="joint2"           slot="1" lower="-1.5"    upper="1.5"/>
+      <xacro:opencr_arm_joint name="joint3"           slot="2" lower="-1.5"    upper="1.4"/>
+      <xacro:opencr_arm_joint name="joint4"           slot="3" lower="-1.7"    upper="2.0"/>
+      <xacro:opencr_arm_joint name="wrist_roll_joint" slot="4" lower="-2.8"    upper="2.8"/>
+      <!-- 6 번째 칸 = 그리퍼 개폐 모터 (ID 15, 모터 각 rad). robot.urdf.xacro 의 가상 관절 (빈 링크) 이라 다른 좌표에 영향 없음.
+           칸이 비면 호스트가 0 을 보내므로 반드시 둔다 — 명령하는 컨트롤러가 없으면 켤 때 위치를 유지.
+           범위 = 펌웨어 config.h 6 번째 칸. gripper_controller 가 이 관절 (모터 각 rad) 을 직접 명령한다.
+           손가락 (gripper_left/right_joint, m) 과의 변환은 미정 ★
+           ⚠ 그리퍼 결합이 0/4095 경계를 지나는 동안 (docs/arm_bench_test_2026-10-26.md 4-4) 은 호스트로 팔 보드를 켜지 않는다 -->
+      <xacro:opencr_arm_joint name="gripper_motor_joint" slot="5" lower="-0.83" upper="1.27"/>
       <sensor name="imu">
         <state_interface name="orientation.x"/>

File: workspace/ros2_ws/src/opencr_hardware/urdf/robot.urdf.xacro (robot description, xacro)
@@ -1,70 +1,35 @@
 <?xml version="1.0"?>
 <!-- 퍽 운반 로봇 URDF (Firmware 팀) — TF 트리 · ros2_control.
-     링크 위치 · 관절 원점은 값이 확정되지 않아 ★ 표시한 자리값이다 (Perception 팀이 센서 장착 위치 제공).
-     형상(visual/collision)은 넣지 않았다. waffle_4wd 메시를 쓰려면 base_link 에 visual 을 추가한다. -->
-<robot name="puckbot" xmlns:xacro="http://www.ros.org/wiki/xacro">
-  <xacro:arg name="wheel_count" default="4"/>   <!-- 주행 펌웨어 WHEEL_COUNT 와 같게 (2026-10-26 가운데 2개 제거) -->
-  <xacro:arg name="use_gripper" default="false"/>
+     몸체 · 관절 · 센서 좌표 · 충돌 · 관성은 CAD 에서 자동 생성한 cartridar_01.urdf 를 그대로 쓴다 (2026-10-26 사용자 1안:
+       4륜 · 바퀴 직결 · RealSense 브래킷 v2 10° · 팔 한계 = 보관함 계획 J1 ±180° · J4 위 124°).
+       FreeCAD TeamRobot/URDF: robot_params.json 수정 → ./run_urdf.sh cartridar_01 → scripts/import_cad_urdf.py 로 가져옴
+       (겉모양 뺌, D435 이름 d435_front/rear → top_camera_front/rear).
+       그 파일은 직접 고치지 않는다.
+     이 파일은 그 위에 ros2_control (opencr.ros2_control.xacro) 과 다른 노드가 쓰는 별칭 좌표만 얹는다.
+     이름 (CAD): 바퀴 wheel_fl/rl/fr/rr_joint · 팔 joint1~4 · wrist_roll_joint · 손가락 gripper_left/right_joint ·
+       센서 top_camera_front/rear_link (+ _optical_frame, D435 깊이 원점 = realsense <camera_name>_link) · lds03_front/rear_link (뒤집어 장착, roll π) · tfmini_link · gripper_camera_link ·
+       imu_link (아래 OpenCR = 주행 보드) · end_effector_link · base_footprint -->
+<robot name="cartridar_01" xmlns:xacro="http://www.ros.org/wiki/xacro">
   <xacro:arg name="ports" default="/dev/ttyACM0,/dev/ttyACM1"/>
   <xacro:arg name="joy_required" default="true"/>
+  <xacro:include filename="$(find opencr_hardware)/urdf/cartridar_01.urdf"/>
   <xacro:include filename="$(find opencr_hardware)/urdf/opencr.ros2_control.xacro"/>
-  <xacro:property name="wheel_count" value="$(arg wheel_count)"/>
-  <xacro:property name="wheel_y" value="0.1585"/>     <!-- 바퀴 중심 |y| (증속벨트 바깥 15 mm 이동 후) ★ -->
-  <xacro:property name="wheel_x" value="0.0925"/>     <!-- 앞바퀴 x (뒤 = 0.025 - 0.0925) -->
-  <xacro:property name="wheel_z" value="0.02625"/>
-  <link name="base_link"/>
-  <xacro:macro name="wheel" params="name x y">
-    <link name="${name}_link"/>
-    <joint name="${name}_joint" type="continuous">
-      <parent link="base_link"/>
-      <child link="${name}_link"/>
-      <origin xyz="${x} ${y} ${wheel_z}" rpy="-1.5708 0 0"/>
-      <axis xyz="0 0 1"/>
-    </joint>
-  </xacro:macro>
-  <xacro:wheel name="wheel_left_front"  x="${wheel_x}"  y="${wheel_y}"/>
-  <xacro:wheel name="wheel_left_rear"   x="${0.025 - wheel_x}" y="${wheel_y}"/>
-  <xacro:wheel name="wheel_right_front" x="${wheel_x}"  y="${-wheel_y}"/>
-  <xacro:wheel name="wheel_right_rear"  x="${0.025 - wheel_x}" y="${-wheel_y}"/>
-  <xacro:if value="${wheel_count == 6}">
-    <xacro:wheel name="wheel_left_mid"  x="0.0125" y="${wheel_y}"/>
-    <xacro:wheel name="wheel_right_mid" x="0.0125" y="${-wheel_y}"/>
-  </xacro:if>
-  <!-- 센서 (정적) ★ 장착 위치 -->
-  <xacro:macro name="fixed_link" params="name parent xyz rpy">
-    <link name="${name}"/>
-    <joint name="${name}_joint" type="fixed">
-      <parent link="${parent}"/>
-      <child link="${name}"/>
-      <origin xyz="${xyz}" rpy="${rpy}"/>
-    </joint>
-  </xacro:macro>
-  <xacro:fixed_link name="imu_link"          parent="base_link" xyz="0 0 0.068" rpy="0 0 0"/>
-  <xacro:fixed_link name="laser_front"       parent="base_link" xyz="0.15 0 0.08" rpy="0 0 0"/>
-  <xacro:fixed_link name="laser_rear"        parent="base_link" xyz="-0.15 0 0.08" rpy="0 0 3.14159"/>
-  <xacro:fixed_link name="camera_front_link" parent="base_link" xyz="0.16 0 0.13" rpy="0 0.35 0"/>
-  <xacro:fixed_link name="camera_rear_link"  parent="base_link" xyz="-0.16 0 0.13" rpy="0 0.35 3.14159"/>
-  <xacro:fixed_link name="arm_base_link"     parent="base_link" xyz="0.087 0 0.111" rpy="0 0 0"/>
-  <!-- 팔 (joint1 요 · joint2~4 피치 · joint5 손목 롤 · gripper_roll) — 길이는 manipulator.yaml 과 같게 ★ -->
-  <xacro:macro name="arm_joint" params="name parent child xyz axis lower upper">
-    <link name="${child}"/>
-    <joint name="${name}" type="revolute">
-      <parent link="${parent}"/>
-      <child link="${child}"/>
-      <origin xyz="${xyz}" rpy="0 0 0"/>
-      <axis xyz="${axis}"/>
-      <limit lower="${lower}" upper="${upper}" effort="4.1" velocity="4.8"/>
-    </joint>
-  </xacro:macro>
-  <xacro:arm_joint name="joint1" parent="arm_base_link" child="link1" xyz="0 0 0.077" axis="0 0 1" lower="-2.8" upper="2.8"/>
-  <xacro:arm_joint name="joint2" parent="link1" child="link2" xyz="0 0 0" axis="0 1 0" lower="-1.8" upper="1.6"/>
-  <xacro:arm_joint name="joint3" parent="link2" child="link3" xyz="0.024 0 0.128" axis="0 1 0" lower="-1.6" upper="1.5"/>
-  <xacro:arm_joint name="joint4" parent="link3" child="link4" xyz="0.124 0 0" axis="0 1 0" lower="-1.8" upper="2.0"/>
-  <xacro:arm_joint name="joint5" parent="link4" child="link5" xyz="0.04 0 0" axis="1 0 0" lower="-2.8" upper="2.8"/>
-  <xacro:arm_joint name="gripper_roll" parent="link5" child="gripper_roll_link" xyz="0.041 0 0" axis="1 0 0" lower="-2.8" upper="2.8"/>
-  <xacro:fixed_link name="arm_camera_link" parent="gripper_roll_link" xyz="0.02 0 0.035" rpy="0 0 0"/>
-  <xacro:fixed_link name="tfmini_link"     parent="gripper_roll_link" xyz="0.02 0 -0.035" rpy="0 0 0"/>
-  <xacro:fixed_link name="tool_link"       parent="gripper_roll_link" xyz="0.086 0 0" rpy="0 0 0"/>
-  <xacro:opencr_ros2_control ports="$(arg ports)" wheel_count="${wheel_count}" use_gripper="$(arg use_gripper)"
-                             joy_required="$(arg joy_required)"/>
+  <!-- 별칭: manipulator_node (Controller 팀) 의 팔 기준 좌표. joint1 축 위, link1 (맨 아래 서보) 높이 — joint2 는 이보다 0.0595 m 위 -->
+  <link name="arm_base_link"/>
+  <joint name="arm_base_link_joint" type="fixed">
+    <parent link="link1"/>
+    <child link="arm_base_link"/>
+    <origin xyz="0.012 0 0" rpy="0 0 0"/>
+  </joint>
+  <!-- 그리퍼 개폐 모터 (팔 6 번째 칸, ID 15) 의 각도 [rad]. 손가락 (gripper_left/right_joint, m) 과의 변환이 정해지기 전까지
+       ros2_control 이 이 관절로 다룬다 (hardware_interface 는 URDF 에 없는 관절을 거부). 빈 링크라 다른 좌표에 영향 없음 -->
+  <link name="gripper_motor_link"/>
+  <joint name="gripper_motor_joint" type="revolute">
+    <parent link="gripper_link"/>
+    <child link="gripper_motor_link"/>
+    <origin xyz="0 0 0" rpy="0 0 0"/>
+    <axis xyz="1 0 0"/>
+    <limit lower="-0.83" upper="1.27" effort="4.1" velocity="4.8"/>
+  </joint>
+  <xacro:opencr_ros2_control ports="$(arg ports)" joy_required="$(arg joy_required)"/>
 </robot>

Commit message: feat: port arm bench firmware (ranges, gripper stall guard, boot PWM check)
Co-Authored-By: Claude Opus 5.5 <noreply@anthropic.com>

File: workspace/ros2_ws/src/opencr_hardware/urdf/opencr.ros2_control.xacro (robot description, xacro)
@@ -51,20 +51,18 @@
       <xacro:opencr_wheel name="wheel_fr_joint" slot="2"/>
       <xacro:opencr_wheel name="wheel_rr_joint" slot="3"/>
-      <!-- 팔 관절 한계 (rad): 호스트가 명령을 이 범위로 자른다 = URDF 한계와 펌웨어 config.h ARM_MIN/MAX_RAD 가 겹치는 구간
-           (펌웨어는 범위 밖 CMD 를 통째로 거부하므로 넘으면 안 됨 - test_robot_description 이 확인).
-           URDF (cartridar_01) 는 보관함 계획 값 J1 ±π · J4 위 2.164 라 joint1 · joint4 는 펌웨어 범위 (±2.8 · 2.0) 에서 잘림.
-           보관함 앞 줄 (J1 최대 2.98 · J4 최대 2.16) 을 쓰려면 펌웨어 범위 · 모터 EEPROM 위치 한계를 넓힌 뒤 (장치 쓰기, 승인) 여기도 넓힘 ★.
-           기구 간섭 (홈 자세 J1 > 137° 면 뒤 프로파일, 롤 180° 근처 J4 > 112° 면 카메라) 은 경로 계획이 피해야 함 -->
-      <xacro:opencr_arm_joint name="joint1"           slot="0" lower="-2.8"    upper="2.8"/>
-      <xacro:opencr_arm_joint name="joint2"           slot="1" lower="-1.5"    upper="1.5"/>
-      <xacro:opencr_arm_joint name="joint3"           slot="2" lower="-1.5"    upper="1.4"/>
-      <xacro:opencr_arm_joint name="joint4"           slot="3" lower="-1.7"    upper="2.0"/>
-      <xacro:opencr_arm_joint name="wrist_roll_joint" slot="4" lower="-2.8"    upper="2.8"/>
-      <!-- 6 번째 칸 = 그리퍼 개폐 모터 (ID 15, 모터 각 rad). robot.urdf.xacro 의 가상 관절 (빈 링크) 이라 다른 좌표에 영향 없음.
+      <!-- 팔 관절 한계 (rad): 호스트가 명령을 이 범위로 자른다. 펌웨어 config.h ARM_MIN/MAX_RAD 안이어야 하고
+           (펌웨어는 범위 밖 CMD 를 통째로 거부 - test_robot_description 이 확인), 로봇 URDF 가 오면 그 <limit> 안이기도 해야 함.
+           2026-10-27 (arm_bench 실물): 펌웨어 범위를 실물에 맞춰 넓힘 (대기 자세 포함 · J1 ±180°) → 여기도 펌웨어 범위 그대로 -->
+      <xacro:opencr_arm_joint name="joint1"           slot="0" lower="-3.14159" upper="3.14159"/>
+      <xacro:opencr_arm_joint name="joint2"           slot="1" lower="-2.14"    upper="1.6"/>
+      <xacro:opencr_arm_joint name="joint3"           slot="2" lower="-1.6"     upper="1.6"/>
+      <xacro:opencr_arm_joint name="joint4"           slot="3" lower="-1.92"    upper="2.0"/>
+      <xacro:opencr_arm_joint name="wrist_roll_joint" slot="4" lower="-2.8"     upper="2.8"/>
+      <!-- 6 번째 칸 = 그리퍼 개폐 모터 (ID 15, 모터 각 rad). 로봇 URDF 에 가상 관절 (빈 링크) 로 둬야 함 (hardware_interface 는 URDF 에 없는 관절을 거부).
            칸이 비면 호스트가 0 을 보내므로 반드시 둔다 — 명령하는 컨트롤러가 없으면 켤 때 위치를 유지.
            범위 = 펌웨어 config.h 6 번째 칸. gripper_controller 가 이 관절 (모터 각 rad) 을 직접 명령한다.
            손가락 (gripper_left/right_joint, m) 과의 변환은 미정 ★
-           ⚠ 그리퍼 결합이 0/4095 경계를 지나는 동안 (docs/arm_bench_test_2026-10-26.md 4-4) 은 호스트로 팔 보드를 켜지 않는다 -->
-      <xacro:opencr_arm_joint name="gripper_motor_joint" slot="5" lower="-0.83" upper="1.27"/>
+           2026-10-27 다시 결합해 0/4095 경계를 지나지 않음 (열림 1550 · 닫힘 2650 tick, 닫을수록 증가). 막힘 보호는 펌웨어 GripGuard -->
+      <xacro:opencr_arm_joint name="gripper_motor_joint" slot="5" lower="-0.7946" upper="0.9541"/>
       <sensor name="imu">
         <state_interface name="orientation.x"/>
